Commit message: Migrate key Params from last successful demo
- Last successful demo code: https://github.com/Monash-Connected-Autonomous-Vehicle/autoware_launch.twizy/tree/23-09-25
- Skipping changes for concatenate_and_time_sync_node.param.yaml since
  that's not needed (see lidar.launch.xml, it relays to
  concatenated/pointcloud)
- Using "velodyne_top_base_link" instead of "velodyne_base_link" for
  sensor_kit.xacro
- Update launch file defaults

File: sensor_kit/twizy_sensor_kit_launch/twizy_sensor_kit_description/urdf/sensor_kit.xacro (robot description, xacro)
@@ -4,6 +4,5 @@
     <xacro:include filename="$(find velodyne_description)/urdf/VLP-16.urdf.xacro"/>
     <!-- <xacro:include filename="$(find vls_description)/urdf/VLS-128.urdf.xacro"/> -->
-    <xacro:include filename="$(find camera_description)/urdf/monocular_camera.xacro"/>
-    <xacro:include filename="$(find imu_description)/urdf/imu.xacro"/>
+    <!-- <xacro:include filename="$(find camera_description)/urdf/monocular_camera.xacro"/> -->
     <xacro:arg name="gpu" default="false"/>
     <xacro:arg name="config_dir" default="$(find twizy_sensor_kit_description)/config"/>
@@ -20,5 +19,5 @@
     <xacro:property name="calibration" value="${xacro.load_yaml('$(arg config_dir)/sensor_kit_calibration.yaml')}"/>
     <!-- lidar -->
-    <xacro:VLP-16 parent="sensor_kit_base_link" name="velodyne_top" topic="/points_raw" hz="10" samples="220" gpu="$(arg gpu)">
+    <xacro:VLP-16 parent="sensor_kit_base_link" name="velodyne" topic="/velodyne_points" hz="10" samples="220" gpu="$(arg gpu)">
       <origin
         xyz="${calibration['sensor_kit_base_link']['velodyne_top_base_link']['x']}
@@ -30,33 +29,4 @@
       />
     </xacro:VLP-16>
-    <!-- camera: Logitech C920-->
-    <xacro:monocular_camera_macro
-      name="camera0/camera"
-      parent="sensor_kit_base_link"
-      namespace=""
-      x="${calibration['sensor_kit_base_link']['camera0/camera_link']['x']}"
-      y="${calibration['sensor_kit_base_link']['camera0/camera_link']['y']}"
-      z="${calibration['sensor_kit_base_link']['camera0/camera_link']['z']}"
-      roll="${calibration['sensor_kit_base_link']['camera0/camera_link']['roll']}"
-      pitch="${calibration['sensor_kit_base_link']['camera0/camera_link']['pitch']}"
-      yaw="${calibration['sensor_kit_base_link']['camera0/camera_link']['yaw']}"
-      fps="30"
-      width="1280"
-      height="720"
-      fov="1.361"
-    />
-    <!-- imu -->
-    <xacro:imu_macro
-      name="sd_imu/imu"
-      parent="sensor_kit_base_link"
-      namespace=""
-      x="${calibration['sensor_kit_base_link']['sd_imu/imu_link']['x']}"
-      y="${calibration['sensor_kit_base_link']['sd_imu/imu_link']['y']}"
-      z="${calibration['sensor_kit_base_link']['sd_imu/imu_link']['z']}"
-      roll="${calibration['sensor_kit_base_link']['sd_imu/imu_link']['roll']}"
-      pitch="${calibration['sensor_kit_base_link']['sd_imu/imu_link']['pitch']}"
-      yaw="${calibration['sensor_kit_base_link']['sd_imu/imu_link']['yaw']}"
-      fps="100"
-    />
   </xacro:macro>
 </robot>

File: vehicle/twizy_vehicle_launch/twizy_vehicle_description/urdf/vehicle.xacro (robot description, xacro)
@@ -1,60 +1,14 @@
 <?xml version="1.0"?>
-<!--
-Copyright (c) 2020 StreetDrone Limited
-Author:  Efimia Panagiotaki
-All rights reserved
--->
-<robot name="sd_twizy" xmlns:xacro="http://www.ros.org/wiki/xacro">
-  <!-- ***************** -->
-  <!-- Imported elements -->
-  <!-- ***************** -->
-  <xacro:include filename="$(find twizy_vehicle_description)/urdf/bases/sd_twizy_body.urdf.xacro" />
-  <xacro:include filename="$(find twizy_vehicle_description)/urdf/wheels/sd_twizy_suspension.urdf.xacro" />
-  <!-- Skipping sensors and using autowares because position updates with sensor_kit calibration files -->
-  <!-- *************** -->
-  <!-- Robots Elements -->
-  <!-- *************** -->
-  <xacro:sd_twizy_base name="sd_twizy"/>
-  <xacro:RL_wheel/>
-  <xacro:RR_wheel/>
-  <xacro:FL_wheel/>
-  <xacro:FR_wheel/>
-  <gazebo>
-    <plugin name="sd_control" filename="libSdControlPlugin.so">
-      <chassis>base_link</chassis>
-      <front_left_wheel>front_left_wheel_joint</front_left_wheel>
-      <front_right_wheel>front_right_wheel_joint</front_right_wheel>
-      <front_left_wheel_steering>front_left_steer_joint</front_left_wheel_steering>
-      <front_right_wheel_steering>front_right_steer_joint</front_right_wheel_steering>
-      <back_left_wheel>rear_left_wheel_joint</back_left_wheel>
-      <back_right_wheel>rear_right_wheel_joint</back_right_wheel>
-      <fl_wheel_steering_p_gain>1e4</fl_wheel_steering_p_gain>
-      <fr_wheel_steering_p_gain>1e4</fr_wheel_steering_p_gain>
-      <fl_wheel_steering_i_gain>0</fl_wheel_steering_i_gain>
-      <fr_wheel_steering_i_gain>0</fr_wheel_steering_i_gain>
-      <fl_wheel_steering_d_gain>3e2</fl_wheel_steering_d_gain>
-      <fr_wheel_steering_d_gain>3e2</fr_wheel_steering_d_gain>
-      <max_speed>22</max_speed>
-      <max_torque>250</max_torque>
-      <front_brake_torque>260</front_brake_torque>
-      <back_brake_torque>260</back_brake_torque>
-      <chassis_aero_force_gain>0.63045</chassis_aero_force_gain>
-    </plugin>
-  </gazebo>
-  <gazebo>
-    <plugin name="p3d" filename="libgazebo_ros_p3d.so">
-      <bodyName>base_link</bodyName>
-      <topicName>base_pose_ground_truth</topicName>
-      <frameName>map</frameName>
-      <updateRate>100.0</updateRate>
-    </plugin>
-  </gazebo>
-  <gazebo>
-    <plugin name="joint_state_publisher" filename="libgazebo_ros_joint_state_publisher.so">
-      <robotNamespace>/sd_twizy</robotNamespace>
-      <jointName>front_left_wheel_joint, front_right_wheel_joint, front_left_steer_joint, front_right_steer_joint, rear_left_wheel_joint, rear_right_wheel_joint</jointName>
-      <updateRate>100.0</updateRate>
-      <alwaysOn>true</alwaysOn>
-    </plugin>
-  </gazebo>
+<robot xmlns:xacro="http://ros.org/wiki/xacro">
+  <!-- load parameter -->
+  <xacro:property name="vehicle_info" value="${xacro.load_yaml('$(find twizy_vehicle_description)/config/vehicle_info.param.yaml')}"/>
+  <!-- vehicle body -->
+  <link name="base_link">
+    <visual>
+      <origin xyz="0 0 0" rpy="${pi/2.0} 0 ${pi/2.0}"/>
+      <geometry>
+        <mesh filename="package://twizy_vehicle_description/mesh/twizy.dae" scale="1 1 1"/>
+      </geometry>
+    </visual>
+  </link>
 </robot>
